Commit message: modified URDF

File: resource/gimbal/urdf/gimbal.urdf (robot description, URDF)
Before this commit: robot Gimbal, 7 links, 6 joints
Links:
- link mount: geometry visual mesh filename=package://resource/meshes/newbase.STL scale=0.001 0.001 0.001

Commit message: modified URDF base

File: resource/gimbal/urdf/gimbal.urdf (robot description, URDF)
Before this commit: robot Gimbal, 7 links, 6 joints
Links:
- link mount: geometry visual mesh filename=package://resource/meshes/base.STL scale=0.001 0.001 0.001
Joints:
- joint yaw: origin xyz=0.06778 0 0.05748 rpy=0 0.78539816339 0 -> xyz=0.12597 0 0.06489 rpy=0 0.78539816339 0

Commit message: added offset from robot imu

File: resource/gimbal/urdf/gimbal.urdf (robot description, URDF)
Before this commit: robot Gimbal, 7 links, 6 joints
Joints:
- joint baseTomount: origin xyz=0 0 0 -> xyz=0.199 0.0 0.0935
